File: ps2_pmod_levelshifter.kicad_pcb (KiCad board)
At the start: 2 copper layers, 35.5 x 23 mm, 4 parts, among them J1 PS/2, J2 PMOD, J3 EXT_POWER

Commit message: update design
Parts:
- moved J1 1.80 mm to (158.8, 91.9)
- moved J2 1.63 mm to (130.0, 85.6)
- moved J3 1.59 mm to (155.5, 100.4)
- moved U1 1.13 mm to (143.6, 91.9)
Connections:
- J1 pad 3: /PS/2_CLK -> VCC_5V
- J1 pad 4: /PS/2_CLK- -> GND_5V
- J1 pad 5: VCC_5V -> /PS/2_CLK
- J1 pad 6: GND_5V -> /PS/2_CLK-
Routing:
- net GND_5V: track 0.00 -> 22.7 mm
- net VCC_3V3: track 0.00 -> 22.4 mm
- net VCC_5V: track 0.00 -> 20.5 mm
- net /PMOD_CLK-: track 0.00 -> 10.2 mm
- net /PMOD_CLK: track 0.00 -> 10.2 mm
- net /PS/2_DATA-: track 0.00 -> 10.2 mm
- net /PS/2_CLK: track 0.00 -> 10.2 mm
- net GND_3V3: track 0.00 -> 10.0 mm
- net /PS/2_DATA: track 0.00 -> 7.92 mm
- net /PS/2_CLK-: track 0.00 -> 7.92 mm
Other:
- board size 35.5 x 23 mm -> 39.9 x 21.1 mm
- board text added: "3V3"
- board text added: "5V"
- board text added: "C1"
- board text added: "C2"
- board text added: "D1"
- board text added: "D2"
- board text added: "GND"

Commit message: update pcb
Parts:
- moved J1 1.55 mm to (158.5, 90.4)
- moved J3 0.28 mm to (155.7, 100.3)
Routing:
- net GND_3V3: track 10.0 -> 18.6 mm
- net /PMOD_DATA-: track 0.00 -> 8.13 mm
- net /PMOD_DATA: track 0.00 -> 8.13 mm
- net VCC_5V: track 20.5 -> 22.8 mm
- net GND_5V: track 22.7 -> 24.2 mm
- net /PS/2_DATA: track 7.92 -> 7.03 mm
- net /PS/2_CLK: track 10.2 -> 10.9 mm
- net /PS/2_DATA-: track 10.2 -> 9.63 mm
Other:
- outline, holes or cut-outs redrawn

Commit message: update design
Routing:
- net /PS/2_CLK-: track 8.30 -> 8.97 mm
- net VCC_5V: track 22.8 -> 23.4 mm
Other:
- board size 39.9 x 21.1 mm -> 39.6 x 21.1 mm
- board text added: "HV"
- board text added: "LV"

Commit message: update design
Parts:
- J3: footprint Connector_PinHeader_2.54mm:PinHeader_1x02_P2.54mm_Vertical -> Connector_PinHeader_2.54mm:PinHeader_1x03_P2.54mm_Vertical
- moved J3 2.55 mm to (158.2, 100.6)
Routing:
- net VCC_3V3: track 22.8 -> 35.7 mm
- net VCC_5V: track 23.4 -> 30.9 mm
- net GND_5V: track 24.1 -> 20.9 mm

Commit message: update design
Other:
- board size 39.6 x 21.1 mm -> 39.6 x 20.8 mm
- board text added: "2025"
- board text added: "PS/2 PMOD"
- board text added: "agtbaskara.com"
Changed lines of the file:
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@@
 		(tags "MINI DIN")
 		(property "Reference" "J1"
-			(at 0 -3.556 90)
+			(at 0 -6.604 90)
 			(layer "F.SilkS")
 			(effects
@@
 		(tags "Through hole pin header THT 1x06 2.54mm single row")
 		(property "Reference" "J2"
-			(at 0 -2.33 0)
+			(at -0.254 14.986 0)
 			(layer "F.SilkS")
 			(effects
@@
 		(layer "Edge.Cuts")
 	)
-	(gr_arc
-		(start 165.862 101.092)
-		(mid 165.415631 102.169631)
-		(end 164.338 102.616)
+	(gr_line
+		(start 165.862 83.058)
+		(end 165.862001 100.838)
 		(stroke
 			(width 0.2)
@@
 		(layer "Edge.Cuts")
 	)
-	(gr_line
-		(start 165.862 83.058)
-		(end 165.862001 101.092)
+	(gr_arc
+		(start 165.862 100.838)
+		(mid 165.415631 101.915631)
+		(end 164.338 102.362)
 		(stroke
 			(width 0.2)
@@
 	)
 	(gr_line
-		(start 127.762 102.616001)
-		(end 164.338 102.616)
+		(start 127.762 102.362)
+		(end 164.338 102.361999)
 		(stroke
 			(width 0.2)
@@
 	)
 	(gr_arc
-		(start 127.762 102.616)
-		(mid 126.684369 102.169631)
-		(end 126.238 101.092)
+		(start 127.762 102.362)
+		(mid 126.684369 101.915631)
+		(end 126.238 100.838)
 		(stroke
 			(width 0.2)
@@
 	)
 	(gr_line
-		(start 126.238 101.092)
+		(start 126.238 100.838)
 		(end 126.238 83.058)
 		(stroke
@@
 		)
 	)
+	(gr_text "2025"
+		(at 149.098 82.804 0)
+		(layer "F.SilkS")
+		(effects
+			(font
+				(size 1.25 1.25)
+				(thickness 0.25)
+				(bold yes)
+			)
+			(justify left)
+		)
+	)
 	(gr_text "D2"
 		(at 131.826 88.138 0)
@@
 		)
 	)
+	(gr_text "agtbaskara.com"
+		(at 132.588 82.804 0)
+		(layer "F.SilkS")
+		(effects
+			(font
+				(size 1.25 1.25)
+				(thickness 0.25)
+				(bold yes)
+			)
+			(justify left)
+		)
+	)
 	(gr_text "LV"
 		(at 140.462 93.218 90)
@@
 	)
 	(gr_text "5V"
-		(at 160.02 101.346 0)
+		(at 160.02 101.092 0)
 		(layer "F.SilkS")
 		(effects
@@
 	)
 	(gr_text "GND"
-		(at 147.066 101.346 0)
+		(at 147.066 101.092 0)
 		(layer "F.SilkS")
 		(effects
+			(font
+				(size 1.25 1.25)
+				(thickness 0.25)
+				(bold yes)
+			)
+			(justify left)
+		)
+	)
+	(gr_text "PS/2 PMOD"
+		(at 133.604 101.092 0)
+		(layer "F.SilkS")
+		(effects

Commit message: update design
Parts:
- J1: footprint r_mini_din:Mini_din6 -> ps2-connector:ps2_mini_din6
- moved J3 0.51 mm to (158.2, 100.1)
- moved J1 0.25 mm to (158.5, 90.2), turned to -90 degrees
- moved J2 0.25 mm to (130.0, 85.3)
- moved U1 0.25 mm to (143.6, 91.7)
Connections:
- J1 pad 3: VCC_5V -> GND_5V
- J1 pad 4: GND_5V -> VCC_5V
Routing:
- net VCC_5V: track 30.9 -> 43.1 mm
- net /PS/2_DATA: track 7.03 -> 15.2 mm
- net GND_5V: track 20.9 -> 15.2 mm
- net /PS/2_CLK-: track 8.97 -> 14.3 mm
- net /PS/2_CLK: track 10.9 -> 5.98 mm
- net /PS/2_DATA-: track 9.63 -> 14.2 mm
Other:
- board size 39.6 x 20.8 mm -> 39.6 x 20.3 mm
